File: DummyLoad.sch (EAGLE design)
At the start: 16 parts, among them IC1 LM358, J1 BINDING-POST, J2 BINDING-POST, Q1 NTE2390-OFFBOARD, SW1 SWITCH-SPDT, X1 SCREW-TERM-2

Commit message: Rough layout
Parts:
- removed X1: SCREW-TERM-2, SaintGimp:SCREW-TERM-2
- added C4: 100uF, SaintGimp:CAP-POL-5-8
- added C5: 2.2uF, SaintGimp:CAP-POL-2.5-5
- added D1: LED, SaintGimp:LED
- added J10, J3, J4, J5, J7, J8, J9: PINHD-1X1, SaintGimp:PINHD-1X1
- added J6: POWERJACK-OFFBRD, SaintGimp:POWERJACK-OFFBRD
- added R10: 47K, SaintGimp:RESISTOR-7.5MM
- added R7: 1M, SaintGimp:RESISTOR-7.5MM
- added R8: 4K7, SaintGimp:RESISTOR-7.5MM
- added R9: (no value), SaintGimp:RESISTOR-7.5MM
- added RV2, RV3: 5K, SaintGimp:POTTRIM
- added SW2: SWITCH-SPDT-OFFBRD, SaintGimp:SWITCH-SPDT-OFFBRD
- added U$1: PANEL-METER-OFFBRD, SaintGimp:PANEL-METER-OFFBRD
- added U1: LP2950, SaintGimp:LP2950
- Q1: value NTE2390-OFFBOARD -> NTE2390; device SaintGimp:NTE2390-OFFBOARD -> SaintGimp:NTE2390
- R3: value 12K -> 180K
- R4: value 3.3K -> 4K7
- R5: value 1R -> 0R1; device SaintGimp:RESISTOR-OFFBOARD -> SaintGimp:RESISTOR-7.5MM
- R6: value 150R -> 68K
- RV1: device SaintGimp:POT-PCB-MOUNT -> SaintGimp:POT-OFFBRD
- SW1: value SWITCH-SPDT -> SWITCH-SPDT-OFFBRD; device SaintGimp:SWITCH-SPDT -> SaintGimp:SWITCH-SPDT-OFFBRD
Connections:
- removed net N$2 (its old number): Q1.GATE, R1.2
- new net +5V: C2.1, C5.+, D1.A, IC1G1.V+, J7.KL, RV1.E, U$1.5V, U1.OUT
- new net GATE: J3.KL, Q1.GATE, R1.2, R7.1
- new net METER: IC1G2.OUT, J10.KL, R6.2, U$1.IN
- new net N$12: R8.1, RV3.E
- new net N$13: IC1G1.+IN, R3.2, SW1.P
- new net N$4: D1.C, R9.1
- new net SENSE: IC1G2.+IN, J4.KL, Q1.SRC, R2.2, R5.2
- net GND: now also C4.-, C5.-, J5.KL, J6.GND, J6.GNDBREAK, J8.KL, J9.KL, R10.1, R7.2, R9.2, RV2.A, RV2.S, RV3.A, RV3.S, U$1.GND, U$1.OUT, U1.GND; no longer IC1G2.+IN, R6.1, X1T2.KL
- net N$1: now also J6.PWR, SW2.P; no longer IC1G2.-IN, IC1G2.OUT
- net N$10: now also R4.2; no longer R3.1, RV1.S
- net N$11: now also RV2.E; no longer R6.2
- net N$3: now also C4.+, SW2.S, U1.IN; no longer Q1.SRC, R2.2, R5.2
- net N$6: now also C3.1, R3.1, RV1.S; no longer R3.2, R4.2, SW1.O
- net N$8: now also IC1G2.-IN, R6.1, R8.2; no longer C2.1, IC1G1.V+, RV1.E, X1T1.KL
- net N$9: now also R10.2, SW1.O; no longer C3.1, IC1G1.+IN, SW1.P
Other:
- note added: "Off-board components, direct-wired together"
- moved on the sheet: C3, IC1G2, J1, J2, Q1, R2, R3, R4, R5, R6, RV1, SW1

Commit message: Second layout pass
Parts:
- R9: value (none) -> 330
- renumbered U$1 to PM1
Connections:
- net +5V: now also PM1.+5V; no longer PM1.5V
- net GATE: now also R1.1; no longer R1.2
- net GND: now also PM1.VOUT; no longer PM1.OUT
- net METER: now also PM1.VIN; no longer PM1.IN
- net N$2: now also R1.2; no longer R1.1
Other:
- moved on the sheet: R1
Changed lines of the file:
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@@
 <part name="C4" library="SaintGimp" deviceset="CAP-POL" device="-5-8" value="100uF"/>
 <part name="C5" library="SaintGimp" deviceset="CAP-POL" device="-2.5-5" value="2.2uF"/>
-<part name="U$1" library="SaintGimp" deviceset="PANEL-METER" device="-OFFBRD"/>
+<part name="PM1" library="SaintGimp" deviceset="PANEL-METER" device="-OFFBRD"/>
 <part name="J7" library="SaintGimp" deviceset="PINHD-1X1" device=""/>
 <part name="GND9" library="SaintGimp" deviceset="GND" device=""/>
@@
 <part name="R8" library="SaintGimp" deviceset="RESISTOR-*" device="7.5MM" value="4K7"/>
 <part name="D1" library="SaintGimp" deviceset="LED" device=""/>
-<part name="R9" library="SaintGimp" deviceset="RESISTOR-*" device="7.5MM"/>
+<part name="R9" library="SaintGimp" deviceset="RESISTOR-*" device="7.5MM" value="330"/>
 <part name="GND12" library="SaintGimp" deviceset="GND" device=""/>
 <part name="R10" library="SaintGimp" deviceset="RESISTOR-*" device="7.5MM" value="47K"/>
@@
 <instance part="IC1" gate="G2" x="53.34" y="106.68"/>
 <instance part="GND2" gate="1" x="38.1" y="50.8"/>
-<instance part="R1" gate="G$1" x="63.5" y="60.96"/>
+<instance part="R1" gate="G$1" x="63.5" y="60.96" rot="R180"/>
 <instance part="R2" gate="G$1" x="63.5" y="45.72"/>
 <instance part="R3" gate="G$1" x="12.7" y="58.42"/>
@@
 <instance part="C4" gate="G$1" x="0" y="81.28"/>
 <instance part="C5" gate="G$1" x="27.94" y="81.28"/>
-<instance part="U$1" gate="G$1" x="121.92" y="91.44"/>
+<instance part="PM1" gate="G$1" x="121.92" y="91.44"/>
 <instance part="J7" gate="G$1" x="78.74" y="93.98" smashed="yes" rot="R180">
 <attribute name="NAME" x="74.93" y="95.631" size="1.778" layer="95"/>
@@
 </segment>
 <segment>
-<pinref part="U$1" gate="G$1" pin="OUT"/>
+<pinref part="PM1" gate="G$1" pin="VOUT"/>
 <wire x1="119.38" y1="88.9" x2="119.38" y2="86.36" width="0.1524" layer="91"/>
 <wire x1="119.38" y1="86.36" x2="101.6" y2="86.36" width="0.1524" layer="91"/>
@@
 </segment>
 <segment>
-<pinref part="U$1" gate="G$1" pin="GND"/>
+<pinref part="PM1" gate="G$1" pin="GND"/>
 <wire x1="124.46" y1="96.52" x2="124.46" y2="78.74" width="0.1524" layer="91"/>
 <wire x1="124.46" y1="78.74" x2="101.6" y2="78.74" width="0.1524" layer="91"/>
@@
 </segment>
 <segment>
-<pinref part="R1" gate="G$1" pin="2"/>
+<pinref part="R1" gate="G$1" pin="1"/>
 <pinref part="J3" gate="G$1" pin="KL"/>
 <label x="78.74" y="60.96" size="1.778" layer="95" xref="yes"/>
@@
 </segment>
 <segment>
-<pinref part="U$1" gate="G$1" pin="5V"/>
+<pinref part="PM1" gate="G$1" pin="+5V"/>
 <wire x1="109.22" y1="96.52" x2="104.14" y2="96.52" width="0.1524" layer="91"/>
 <wire x1="104.14" y1="96.52" x2="104.14" y2="93.98" width="0.1524" layer="91"/>
@@
 <net name="N$2" class="0">
 <segment>
-<pinref part="R1" gate="G$1" pin="1"/>
+<pinref part="R1" gate="G$1" pin="2"/>
 <pinref part="IC1" gate="G1" pin="OUT"/>
 <wire x1="58.42" y1="60.96" x2="53.34" y2="60.96" width="0.1524" layer="91"/>
@@
 <net name="METER" class="0">
 <segment>
-<pinref part="U$1" gate="G$1" pin="IN"/>
+<pinref part="PM1" gate="G$1" pin="VIN"/>
 <wire x1="114.3" y1="88.9" x2="106.68" y2="88.9" width="0.1524" layer="91"/>
 <label x="104.14" y="106.68" size="1.778" layer="95" rot="R180" xref="yes"/>

Commit message: Tweak values
Parts:
- removed R7: 1M, SaintGimp:RESISTOR-7.5MM
- C1: value 0.1uF -> 22nF
- C4: device SaintGimp:CAP-POL-5-8 -> SaintGimp:CAP-POL-2.5-5
- R1: value 100R -> 470R
Connections:
- net GATE: no longer R7.1
- net GND: no longer R7.2
Changed lines of the file:
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@@
 <?xml version="1.0" encoding="utf-8"?>
 <!DOCTYPE eagle SYSTEM "eagle.dtd">
-<eagle version="7.2.0">
+<eagle version="7.4.0">
 <drawing>
 <settings>
@@
 <layer number="56" name="wert" color="7" fill="1" visible="no" active="no"/>
 <layer number="57" name="tCAD" color="7" fill="1" visible="no" active="no"/>
+<layer number="59" name="tCarbon" color="7" fill="1" visible="no" active="no"/>
+<layer number="60" name="bCarbon" color="7" fill="1" visible="no" active="no"/>
 <layer number="90" name="Modules" color="5" fill="1" visible="yes" active="yes"/>
 <layer number="91" name="Nets" color="2" fill="1" visible="yes" active="yes"/>
@@
 <layer number="113" name="IDFDebug" color="7" fill="1" visible="yes" active="yes"/>
 <layer number="116" name="Patch_BOT" color="9" fill="4" visible="yes" active="yes"/>
+<layer number="118" name="Rect_Pads" color="7" fill="1" visible="no" active="no"/>
 <layer number="121" name="_tsilk" color="7" fill="1" visible="yes" active="yes"/>
 <layer number="122" name="_bsilk" color="7" fill="1" visible="yes" active="yes"/>
@@
 <layer number="127" name="_tValues" color="7" fill="1" visible="yes" active="yes"/>
 <layer number="128" name="_bValues" color="7" fill="1" visible="yes" active="yes"/>
+<layer number="129" name="Mask" color="7" fill="1" visible="yes" active="yes"/>
 <layer number="131" name="tAdjust" color="7" fill="1" visible="yes" active="yes"/>
 <layer number="132" name="bAdjust" color="7" fill="1" visible="yes" active="yes"/>
@@
 <layer number="230" name="230bmp" color="7" fill="1" visible="yes" active="yes"/>
 <layer number="231" name="231bmp" color="7" fill="1" visible="yes" active="yes"/>
+<layer number="232" name="Eagle3D_PG2" color="7" fill="1" visible="no" active="no"/>
+<layer number="233" name="Eagle3D_PG3" color="7" fill="1" visible="no" active="no"/>
 <layer number="248" name="Housing" color="7" fill="1" visible="yes" active="yes"/>
 <layer number="249" name="Edge" color="7" fill="1" visible="yes" active="yes"/>
@@
 <part name="IC1" library="SaintGimp" deviceset="LM358" device=""/>
 <part name="GND2" library="SaintGimp" deviceset="GND" device=""/>
-<part name="R1" library="SaintGimp" deviceset="RESISTOR-*" device="7.5MM" value="100R"/>
+<part name="R1" library="SaintGimp" deviceset="RESISTOR-*" device="7.5MM" value="470R"/>
 <part name="R2" library="SaintGimp" deviceset="RESISTOR-*" device="7.5MM" value="1K"/>
 <part name="R3" library="SaintGimp" deviceset="RESISTOR-*" device="7.5MM" value="180K"/>
 <part name="Q1" library="SaintGimp" deviceset="NTE2390" device="" value="NTE2390"/>
 <part name="R5" library="SaintGimp" deviceset="RESISTOR-*" device="7.5MM" value="0R1"/>
-<part name="C1" library="SaintGimp" deviceset="CAPACITOR-*" device="5MM" value="0.1uF"/>
+<part name="C1" library="SaintGimp" deviceset="CAPACITOR-*" device="5MM" value="22nF"/>
 <part name="GND3" library="SaintGimp" deviceset="GND" device=""/>
 <part name="J1" library="SaintGimp" deviceset="BINDING-POST" device=""/>
@@
 <part name="J6" library="SaintGimp" deviceset="POWERJACK" device="-OFFBRD"/>
 <part name="U1" library="SaintGimp" deviceset="LP2950" device=""/>
-<part name="C4" library="SaintGimp" deviceset="CAP-POL" device="-5-8" value="100uF"/>
+<part name="C4" library="SaintGimp" deviceset="CAP-POL" device="-2.5-5" value="100uF"/>
 <part name="C5" library="SaintGimp" deviceset="CAP-POL" device="-2.5-5" value="2.2uF"/>
 <part name="PM1" library="SaintGimp" deviceset="PANEL-METER" device="-OFFBRD"/>
@@
 <part name="GND1" library="SaintGimp" deviceset="GND" device=""/>
 <part name="J10" library="SaintGimp" deviceset="PINHD-1X1" device=""/>
-<part name="R7" library="SaintGimp" deviceset="RESISTOR-*" device="7.5MM" value="1M"/>
-<part name="GND11" library="SaintGimp" deviceset="GND" device=""/>
 <part name="SW2" library="SaintGimp" deviceset="SWITCH-SPDT" device="-OFFBRD"/>
 <part name="R8" library="SaintGimp" deviceset="RESISTOR-*" device="7.5MM" value="4K7"/>
@@
 <attribute name="NAME" x="72.39" y="108.331" size="1.778" layer="95"/>
 </instance>
-<instance part="R7" gate="G$1" x="71.12" y="66.04" rot="R90"/>
-<instance part="GND11" gate="1" x="73.66" y="71.12" rot="R90"/>
 <instance part="SW2" gate="G$1" x="-7.62" y="86.36"/>
 <instance part="R8" gate="G$1" x="40.64" y="96.52"/>
@@
 </segment>
 <segment>
-<pinref part="R7" gate="G$1" pin="2"/>
-<pinref part="GND11" gate="1" pin="GND"/>
-</segment>
-<segment>
 <pinref part="RV3" gate="G$1" pin="A"/>
 <pinref part="GND1" gate="1" pin="GND"/>
@@
 <pinref part="J3" gate="G$1" pin="KL"/>
 <label x="78.74" y="60.96" size="1.778" layer="95" xref="yes"/>
-<wire x1="73.66" y1="60.96" x2="71.12" y2="60.96" width="0.1524" layer="91"/>
-<pinref part="R7" gate="G$1" pin="1"/>
-<wire x1="71.12" y1="60.96" x2="68.58" y2="60.96" width="0.1524" layer="91"/>
-<junction x="71.12" y="60.96"/>
+<wire x1="73.66" y1="60.96" x2="68.58" y2="60.96" width="0.1524" layer="91"/>
 </segment>
 </net>

Commit message: Clean up layout
Parts:
- C4: device SaintGimp:CAP-POL-2.5-5 -> SaintGimp:CAP-POL-2.5-6
Changed lines of the file:
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@@
 <part name="J6" library="SaintGimp" deviceset="POWERJACK" device="-OFFBRD"/>
 <part name="U1" library="SaintGimp" deviceset="LP2950" device=""/>
-<part name="C4" library="SaintGimp" deviceset="CAP-POL" device="-2.5-5" value="100uF"/>
-<part name="C5" library="SaintGimp" deviceset="CAP-POL" device="-2.5-5" value="2.2uF"/>
+<part name="C4" library="SaintGimp" deviceset="CAP-POL-*" device="2.5-6" value="100uF"/>
+<part name="C5" library="SaintGimp" deviceset="CAP-POL-*" device="2.5-5" value="2.2uF"/>
 <part name="PM1" library="SaintGimp" deviceset="PANEL-METER" device="-OFFBRD"/>
 <part name="J7" library="SaintGimp" deviceset="PINHD-1X1" device=""/>
@@
 <instance part="RV2" gate="G$1" x="12.7" y="33.02"/>
 <instance part="R4" gate="G$1" x="12.7" y="45.72" rot="R90"/>
-<instance part="J3" gate="G$1" x="78.74" y="60.96" smashed="yes" rot="R180">
+<instance part="J3" gate="1" x="78.74" y="60.96" smashed="yes" rot="R180">
 <attribute name="NAME" x="74.93" y="62.611" size="1.778" layer="95"/>
 </instance>
-<instance part="J4" gate="G$1" x="76.2" y="45.72" smashed="yes" rot="R180">
+<instance part="J4" gate="1" x="76.2" y="45.72" smashed="yes" rot="R180">
 <attribute name="NAME" x="72.39" y="47.371" size="1.778" layer="95"/>
 </instance>
 <instance part="GND4" gate="1" x="68.58" y="30.48" rot="R270"/>
-<instance part="J5" gate="G$1" x="78.74" y="30.48" smashed="yes" rot="R180">
+<instance part="J5" gate="1" x="78.74" y="30.48" smashed="yes" rot="R180">
 <attribute name="NAME" x="74.93" y="32.131" size="1.778" layer="95"/>
 </instance>
@@
 <instance part="C5" gate="G$1" x="27.94" y="81.28"/>
 <instance part="PM1" gate="G$1" x="121.92" y="91.44"/>
-<instance part="J7" gate="G$1" x="78.74" y="93.98" smashed="yes" rot="R180">
+<instance part="J7" gate="1" x="78.74" y="93.98" smashed="yes" rot="R180">
 <attribute name="NAME" x="74.93" y="95.631" size="1.778" layer="95"/>
 </instance>
 <instance part="GND9" gate="1" x="68.58" y="78.74" rot="R270"/>
-<instance part="J8" gate="G$1" x="78.74" y="78.74" smashed="yes" rot="R180">
+<instance part="J8" gate="1" x="78.74" y="78.74" smashed="yes" rot="R180">
 <attribute name="NAME" x="74.93" y="80.391" size="1.778" layer="95"/>
 </instance>
 <instance part="GND10" gate="1" x="68.58" y="86.36" rot="R270"/>
-<instance part="J9" gate="G$1" x="78.74" y="86.36" smashed="yes" rot="R180">
+<instance part="J9" gate="1" x="78.74" y="86.36" smashed="yes" rot="R180">
 <attribute name="NAME" x="74.93" y="88.011" size="1.778" layer="95"/>
 </instance>
@@
 <instance part="RV3" gate="G$1" x="25.4" y="96.52" rot="R270"/>
 <instance part="GND1" gate="1" x="15.24" y="96.52" rot="R270"/>
-<instance part="J10" gate="G$1" x="76.2" y="106.68" smashed="yes" rot="R180">
+<instance part="J10" gate="1" x="76.2" y="106.68" smashed="yes" rot="R180">
 <attribute name="NAME" x="72.39" y="108.331" size="1.778" layer="95"/>
 </instance>
@@
 <segment>
 <pinref part="GND4" gate="1" pin="GND"/>
-<pinref part="J5" gate="G$1" pin="KL"/>
+<pinref part="J5" gate="1" pin="KL"/>
 <wire x1="71.12" y1="30.48" x2="73.66" y2="30.48" width="0.1524" layer="91"/>
 <label x="78.74" y="30.48" size="1.778" layer="95" xref="yes"/>
@@
 <segment>
 <pinref part="GND9" gate="1" pin="GND"/>
-<pinref part="J8" gate="G$1" pin="KL"/>
+<pinref part="J8" gate="1" pin="KL"/>
 <wire x1="71.12" y1="78.74" x2="73.66" y2="78.74" width="0.1524" layer="91"/>
 <label x="78.74" y="78.74" size="1.778" layer="95" xref="yes"/>
@@
 <segment>
 <pinref part="GND10" gate="1" pin="GND"/>
-<pinref part="J9" gate="G$1" pin="KL"/>
+<pinref part="J9" gate="1" pin="KL"/>
 <wire x1="71.12" y1="86.36" x2="73.66" y2="86.36" width="0.1524" layer="91"/>
 <label x="78.74" y="86.36" size="1.778" layer="95" xref="yes"/>
@@
 <segment>
 <pinref part="R1" gate="G$1" pin="1"/>
-<pinref part="J3" gate="G$1" pin="KL"/>
+<pinref part="J3" gate="1" pin="KL"/>
 <label x="78.74" y="60.96" size="1.778" layer="95" xref="yes"/>
 <wire x1="73.66" y1="60.96" x2="68.58" y2="60.96" width="0.1524" layer="91"/>
@@
 <junction x="27.94" y="83.82"/>
 <label x="78.74" y="93.98" size="1.778" layer="95" xref="yes"/>
-<pinref part="J7" gate="G$1" pin="KL"/>
+<pinref part="J7" gate="1" pin="KL"/>
 <wire x1="73.66" y1="93.98" x2="45.72" y2="93.98" width="0.1524" layer="91"/>
 <wire x1="45.72" y1="93.98" x2="45.72" y2="83.82" width="0.1524" layer="91"/>
@@
 <segment>
 <pinref part="R2" gate="G$1" pin="2"/>
-<pinref part="J4" gate="G$1" pin="KL"/>
+<pinref part="J4" gate="1" pin="KL"/>
 <wire x1="71.12" y1="45.72" x2="68.58" y2="45.72" width="0.1524" layer="91"/>
 <label x="76.2" y="45.72" size="1.778" layer="95" xref="yes"/>
@@
 <pinref part="IC1" gate="G2" pin="OUT"/>
 <pinref part="R6" gate="G$1" pin="2"/>
-<pinref part="J10" gate="G$1" pin="KL"/>
+<pinref part="J10" gate="1" pin="KL"/>
 <junction x="71.12" y="106.68"/>
 <label x="76.2" y="106.68" size="1.778" layer="95" xref="yes"/>

Commit message: Design updates
Parts:
- removed J1, J2: BINDING-POST, SaintGimp:BINDING-POST
- removed PM1: PANEL-METER-OFFBRD, SaintGimp:PANEL-METER-OFFBRD
- removed Q1: NTE2390, SaintGimp:NTE2390
- added R11, R12, R13, R14, R15, R16, R17, R18, R7: 1R, SaintGimp:RESISTOR-7.5MM
- R5: value 0R1 -> 1R
Connections:
- removed net N$7: J2.1, Q1.DRN
- net +5V: no longer PM1.+5V
- net GATE: no longer Q1.GATE
- net GND: now also R11.2, R12.2, R13.2, R14.2, R15.2, R16.2, R17.2, R18.2, R5.2, R7.2; no longer J1.1, PM1.GND, PM1.VOUT, R5.1
- net METER: no longer PM1.VIN
- net SENSE: now also R11.1, R12.1, R13.1, R14.1, R15.1, R16.1, R17.1, R18.1, R5.1, R7.1; no longer Q1.SRC, R5.2
Other:
- note removed: "Off-board components, direct-wired together"
- moved on the sheet: J4, J5, R5
