File: DummyLoad.sch (EAGLE design)
At the start: 39 parts, among them IC1 LM358, J10 PINHD-1X1, J3 PINHD-1X1, J4 PINHD-1X1, J5 PINHD-1X1, J6 POWERJACK-OFFBRD, J7 PINHD-1X1, J8 PINHD-1X1, J9 PINHD-1X1, SW1 SWITCH-SPDT-OFFBRD, SW2 SWITCH-SPDT-OFFBRD, U1 LP2950

Commit message: Tweaked layout
Parts:
- removed J6: POWERJACK-OFFBRD, SaintGimp:POWERJACK-OFFBRD
- removed R10: 47K, SaintGimp:RESISTOR-7.5MM
- removed SW1, SW2: SWITCH-SPDT-OFFBRD, SaintGimp:SWITCH-SPDT-OFFBRD
- added J1: PINHD-1X2, SaintGimp:PINHD-1X2
- D1: value LED -> LED-5MM; device SaintGimp:LED -> SaintGimp:LED-5MM
- IC1: value LM358 -> MCP6022; device SaintGimp:LM358 -> SaintGimp:MCP6022
- R9: value 330 -> 470
Connections:
- removed net N$1: J6.PWR, SW2.P
- removed net N$10: R4.2, SW1.S
- removed net N$9: R10.2, SW1.O
- net GND: now also J12.KL; no longer J6.GND, J6.GNDBREAK, R10.1
- net N$13: now also R4.2; no longer SW1.P
- net N$3: now also J11.KL; no longer SW2.S
Other:
- moved on the sheet: R4, RV2
Changed lines of the file:
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@@
 <?xml version="1.0" encoding="utf-8"?>
 <!DOCTYPE eagle SYSTEM "eagle.dtd">
-<eagle version="7.4.0">
+<eagle version="7.7.0">
 <drawing>
 <settings>
@@
 <layer number="112" name="tSilk" color="7" fill="1" visible="yes" active="yes"/>
 <layer number="113" name="IDFDebug" color="7" fill="1" visible="yes" active="yes"/>
+<layer number="114" name="FRNTMAAT1" color="7" fill="1" visible="yes" active="yes"/>
+<layer number="115" name="FRNTMAAT2" color="7" fill="1" visible="yes" active="yes"/>
 <layer number="116" name="Patch_BOT" color="9" fill="4" visible="yes" active="yes"/>
+<layer number="117" name="BACKMAAT1" color="7" fill="1" visible="yes" active="yes"/>
 <layer number="118" name="Rect_Pads" color="7" fill="1" visible="no" active="no"/>
+<layer number="119" name="KAP_TEKEN" color="7" fill="1" visible="yes" active="yes"/>
+<layer number="120" name="KAP_MAAT1" color="7" fill="1" visible="yes" active="yes"/>
 <layer number="121" name="_tsilk" color="7" fill="1" visible="yes" active="yes"/>
 <layer number="122" name="_bsilk" color="7" fill="1" visible="yes" active="yes"/>
@@
 <layer number="128" name="_bValues" color="7" fill="1" visible="yes" active="yes"/>
 <layer number="129" name="Mask" color="7" fill="1" visible="yes" active="yes"/>
+<layer number="130" name="SMDSTROOK" color="7" fill="1" visible="yes" active="yes"/>
 <layer number="131" name="tAdjust" color="7" fill="1" visible="yes" active="yes"/>
 <layer number="132" name="bAdjust" color="7" fill="1" visible="yes" active="yes"/>
+<layer number="133" name="bottom_silk" color="7" fill="1" visible="yes" active="yes"/>
 <layer number="144" name="Drill_legend" color="7" fill="1" visible="yes" active="yes"/>
 <layer number="150" name="Notes" color="7" fill="1" visible="yes" active="yes"/>
@@
 </classes>
 <parts>
-<part name="IC1" library="SaintGimp" deviceset="LM358" device=""/>
+<part name="IC1" library="SaintGimp" deviceset="MCP6022" device=""/>
 <part name="GND2" library="SaintGimp" deviceset="GND" device=""/>
 <part name="R1" library="SaintGimp" deviceset="RESISTOR-*" device="7.5MM" value="470R"/>
@@
 <part name="GND7" library="SaintGimp" deviceset="GND" device=""/>
 <part name="GND8" library="SaintGimp" deviceset="GND" device=""/>
-<part name="SW1" library="SaintGimp" deviceset="SWITCH-SPDT" device="-OFFBRD" value="SWITCH-SPDT-OFFBRD"/>
 <part name="RV2" library="SaintGimp" deviceset="POT" device="TRIM" value="5K"/>
 <part name="R4" library="SaintGimp" deviceset="RESISTOR-*" device="7.5MM" value="4K7"/>
@@
 <part name="GND4" library="SaintGimp" deviceset="GND" device=""/>
 <part name="J5" library="SaintGimp" deviceset="PINHD-1X1" device=""/>
-<part name="J6" library="SaintGimp" deviceset="POWERJACK" device="-OFFBRD"/>
 <part name="U1" library="SaintGimp" deviceset="LP2950" device=""/>
 <part name="C4" library="SaintGimp" deviceset="CAP-POL-*" device="2.5-6" value="100uF"/>
@@
 <part name="GND1" library="SaintGimp" deviceset="GND" device=""/>
 <part name="J10" library="SaintGimp" deviceset="PINHD-1X1" device=""/>
-<part name="SW2" library="SaintGimp" deviceset="SWITCH-SPDT" device="-OFFBRD"/>
 <part name="R8" library="SaintGimp" deviceset="RESISTOR-*" device="7.5MM" value="4K7"/>
-<part name="D1" library="SaintGimp" deviceset="LED" device=""/>
-<part name="R9" library="SaintGimp" deviceset="RESISTOR-*" device="7.5MM" value="330"/>
+<part name="D1" library="SaintGimp" deviceset="LED-*" device="5MM"/>
+<part name="R9" library="SaintGimp" deviceset="RESISTOR-*" device="7.5MM" value="470"/>
 <part name="GND12" library="SaintGimp" deviceset="GND" device=""/>
-<part name="R10" library="SaintGimp" deviceset="RESISTOR-*" device="7.5MM" value="47K"/>
-<part name="GND13" library="SaintGimp" deviceset="GND" device=""/>
 <part name="R5" library="SaintGimp" deviceset="RESISTOR-*" device="7.5MM" value="1R"/>
 <part name="R7" library="SaintGimp" deviceset="RESISTOR-*" device="7.5MM" value="1R"/>
@@
 <part name="R17" library="SaintGimp" deviceset="RESISTOR-*" device="7.5MM" value="1R"/>
 <part name="R18" library="SaintGimp" deviceset="RESISTOR-*" device="7.5MM" value="1R"/>
+<part name="J1" library="SaintGimp" deviceset="PINHD-1X2" device=""/>
 </parts>
 <sheets>
@@
 <instance part="R3" gate="G$1" x="12.7" y="58.42"/>
 <instance part="C1" gate="G$1" x="53.34" y="53.34"/>
-<instance part="GND3" gate="1" x="12.7" y="22.86"/>
+<instance part="GND3" gate="1" x="20.32" y="27.94"/>
 <instance part="C2" gate="G$1" x="43.18" y="71.12" rot="R90"/>
 <instance part="GND5" gate="1" x="48.26" y="71.12" rot="R90"/>
@@
 <instance part="GND7" gate="1" x="2.54" y="48.26"/>
 <instance part="GND8" gate="1" x="-10.16" y="73.66"/>
-<instance part="SW1" gate="G$1" x="22.86" y="53.34" rot="R270"/>
-<instance part="RV2" gate="G$1" x="12.7" y="33.02"/>
-<instance part="R4" gate="G$1" x="12.7" y="45.72" rot="R90"/>
+<instance part="RV2" gate="G$1" x="20.32" y="38.1"/>
+<instance part="R4" gate="G$1" x="20.32" y="50.8" rot="R90"/>
 <instance part="J3" gate="1" x="78.74" y="60.96" smashed="yes" rot="R180">
 <attribute name="NAME" x="74.93" y="62.611" size="1.778" layer="95"/>
@@
 <attribute name="NAME" x="121.031" y="26.67" size="1.778" layer="95" rot="R270"/>
 </instance>
-<instance part="J6" gate="G$1" x="-27.94" y="81.28"/>
 <instance part="U1" gate="G$1" x="15.24" y="81.28"/>
 <instance part="C4" gate="G$1" x="0" y="81.28"/>
@@
 <attribute name="NAME" x="72.39" y="108.331" size="1.778" layer="95"/>
 </instance>
-<instance part="SW2" gate="G$1" x="-7.62" y="86.36"/>
 <instance part="R8" gate="G$1" x="40.64" y="96.52"/>
 <instance part="D1" gate="1" x="50.8" y="83.82" rot="R90"/>
 <instance part="R9" gate="G$1" x="58.42" y="78.74" rot="R270"/>
 <instance part="GND12" gate="1" x="58.42" y="71.12"/>
-<instance part="R10" gate="G$1" x="22.86" y="45.72" rot="R90"/>
-<instance part="GND13" gate="1" x="22.86" y="38.1"/>
 <instance part="R5" gate="G$1" x="114.3" y="109.22"/>
 <instance part="R7" gate="G$1" x="114.3" y="101.6"/>
@@
 <instance part="R17" gate="G$1" x="114.3" y="48.26"/>
 <instance part="R18" gate="G$1" x="114.3" y="40.64"/>
+<instance part="J1" gate="1" x="-20.32" y="83.82"/>
+<instance part="J1" gate="2" x="-20.32" y="76.2"/>
 </instances>
 <busses>
@@
 <wire x1="27.94" y1="76.2" x2="15.24" y2="76.2" width="0.1524" layer="91"/>
 <junction x="15.24" y="76.2"/>
-<wire x1="-10.16" y1="76.2" x2="-20.32" y2="76.2" width="0.1524" layer="91"/>
+<wire x1="-10.16" y1="76.2" x2="-15.24" y2="76.2" width="0.1524" layer="91"/>
 <junction x="-10.16" y="76.2"/>
-<pinref part="J6" gate="G$1" pin="GND"/>
-<pinref part="J6" gate="G$1" pin="GNDBREAK"/>
-<wire x1="-20.32" y1="81.28" x2="-20.32" y2="78.74" width="0.1524" layer="91"/>
-<wire x1="-20.32" y1="76.2" x2="-20.32" y2="78.74" width="0.1524" layer="91"/>
-<junction x="-20.32" y="78.74"/>
+<pinref part="J1" gate="2" pin="KL"/>
 </segment>
 <segment>
@@
 <pinref part="GND3" gate="1" pin="GND"/>
 <pinref part="RV2" gate="G$1" pin="S"/>
-<wire x1="17.78" y1="33.02" x2="17.78" y2="25.4" width="0.1524" layer="91"/>
-<wire x1="17.78" y1="25.4" x2="12.7" y2="25.4" width="0.1524" layer="91"/>
-<junction x="12.7" y="25.4"/>
+<wire x1="25.4" y1="38.1" x2="25.4" y2="30.48" width="0.1524" layer="91"/>
+<wire x1="25.4" y1="30.48" x2="20.32" y2="30.48" width="0.1524" layer="91"/>
+<junction x="20.32" y="30.48"/>
 </segment>
 <segment>
 <pinref part="R9" gate="G$1" pin="2"/>
 <pinref part="GND12" gate="1" pin="GND"/>
-</segment>
-<segment>
-<pinref part="R10" gate="G$1" pin="1"/>
-<pinref part="GND13" gate="1" pin="GND"/>
 </segment>
 <segment>
@@
 <pinref part="C4" gate="G$1" pin="+"/>
 <wire x1="0" y1="83.82" x2="7.62" y2="83.82" width="0.1524" layer="91"/>
-<pinref part="SW2" gate="G$1" pin="S"/>
-<wire x1="0" y1="83.82" x2="-5.08" y2="83.82" width="0.1524" layer="91"/>
+<pinref part="J1" gate="1" pin="KL"/>
+<wire x1="0" y1="83.82" x2="-15.24" y2="83.82" width="0.1524" layer="91"/>
 <junction x="0" y="83.82"/>
 </segment>
@@
 </segment>
 </net>
-<net name="N$1" class="0">
-<segment>
-<pinref part="SW2" gate="G$1" pin="P"/>
-<pinref part="J6" gate="G$1" pin="PWR"/>
-<wire x1="-12.7" y1="86.36" x2="-20.32" y2="86.36" width="0.1524" layer="91"/>
-<wire x1="-20.32" y1="86.36" x2="-20.32" y2="83.82" width="0.1524" layer="91"/>
-</segment>
-</net>
 <net name="N$8" class="0">
 <segment>
@@
 </segment>
 </net>
-<net name="N$9" class="0">
-<segment>
-<pinref part="SW1" gate="G$1" pin="O"/>
-<pinref part="R10" gate="G$1" pin="2"/>
-<wire x1="22.86" y1="50.8" x2="25.4" y2="50.8" width="0.1524" layer="91"/>
-</segment>
-</net>
-<net name="N$10" class="0">
-<segment>
-<pinref part="SW1" gate="G$1" pin="S"/>
+<net name="N$13" class="0">
+<segment>
+<pinref part="IC1" gate="G1" pin="+IN"/>
+<wire x1="33.02" y1="58.42" x2="20.32" y2="58.42" width="0.1524" layer="91"/>
+<pinref part="R3" gate="G$1" pin="2"/>
 <pinref part="R4" gate="G$1" pin="2"/>
-<wire x1="20.32" y1="50.8" x2="12.7" y2="50.8" width="0.1524" layer="91"/>
-</segment>
-</net>
-<net name="N$13" class="0">
-<segment>
-<pinref part="IC1" gate="G1" pin="+IN"/>
-<pinref part="SW1" gate="G$1" pin="P"/>
-<wire x1="33.02" y1="58.42" x2="22.86" y2="58.42" width="0.1524" layer="91"/>
-<pinref part="R3" gate="G$1" pin="2"/>
-<wire x1="22.86" y1="58.42" x2="17.78" y2="58.42" width="0.1524" layer="91"/>
-<junction x="22.86" y="58.42"/>
-</segment>
-</net>
+<wire x1="20.32" y1="58.42" x2="17.78" y2="58.42" width="0.1524" layer="91"/>
+<wire x1="20.32" y1="55.88" x2="20.32" y2="58.42" width="0.1524" layer="91"/>
+<junction x="20.32" y="58.42"/>
+</segment>
+</net>
